File: ucruler.brd (EAGLE design)
At the start: 200 x 32 mm, 27 parts

Commit message: thermal resistance for vias
Parts:
- added E$28: (no value), ucruler:SILK-TABLE-THVIA
Changed lines of the file:
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@@
 <layer number="21" name="tPlace" color="7" fill="1" visible="no" active="yes"/>
 <layer number="22" name="bPlace" color="7" fill="1" visible="yes" active="yes"/>
-<layer number="23" name="tOrigins" color="15" fill="1" visible="no" active="yes"/>
+<layer number="23" name="tOrigins" color="15" fill="1" visible="yes" active="yes"/>
 <layer number="24" name="bOrigins" color="15" fill="1" visible="yes" active="yes"/>
 <layer number="25" name="tNames" color="7" fill="1" visible="no" active="yes"/>
@@
 <element name="E$22" library="ucruler" package="SILK-FONT" value="" x="141" y="29" rot="MR270"/>
 <element name="E$23" library="ucruler" package="SILK-TABLE-SMDR" value="" x="193" y="29" rot="MR0"/>
+<element name="E$28" library="ucruler" package="SILK-TABLE-THVIA" value="" x="131" y="27" rot="MR0"/>
 </elements>
 <signals>

Commit message: wrong arrow direction on npn transistor fixed
Parts:
- added E$29: (no value), ucruler:SILK-TABLE-MM-MIL
Other:
- board text removed: "[mm] [mil] 0,10 4 0,15 6 0,20 8 0,30 12 0,5 20 1,0 39 1,5 59 2,0 79"
Changed lines of the file:
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@@
 <layer number="19" name="Unrouted" color="6" fill="1" visible="yes" active="yes"/>
 <layer number="20" name="Dimension" color="15" fill="1" visible="yes" active="yes"/>
-<layer number="21" name="tPlace" color="7" fill="1" visible="no" active="yes"/>
+<layer number="21" name="tPlace" color="7" fill="1" visible="yes" active="yes"/>
 <layer number="22" name="bPlace" color="7" fill="1" visible="yes" active="yes"/>
-<layer number="23" name="tOrigins" color="15" fill="1" visible="yes" active="yes"/>
+<layer number="23" name="tOrigins" color="15" fill="1" visible="no" active="yes"/>
 <layer number="24" name="bOrigins" color="15" fill="1" visible="yes" active="yes"/>
 <layer number="25" name="tNames" color="7" fill="1" visible="no" active="yes"/>
@@
 <rectangle x1="29" y1="4" x2="37" y2="19" layer="29"/>
 <rectangle x1="13.25" y1="4" x2="20.75" y2="27" layer="29"/>
-<text x="83" y="27" size="1.2" layer="21" align="top-left">[mm] [mil]
-0,10   4
-0,15   6
-0,20   8
-0,30  12
-0,5   20
-1,0   39
-1,5   59
-2,0   79
-</text>
 <text x="194.75" y="3" size="1.5" layer="22" rot="MR90" align="top-left">Owner</text>
 <hole x="198.755" y="1.905" drill="0.8"/>
@@
 <element name="E$23" library="ucruler" package="SILK-TABLE-SMDR" value="" x="193" y="29" rot="MR0"/>
 <element name="E$28" library="ucruler" package="SILK-TABLE-THVIA" value="" x="131" y="27" rot="MR0"/>
+<element name="E$29" library="ucruler" package="SILK-TABLE-MM-MIL" value="" x="121" y="29" rot="MR0"/>
 </elements>
 <signals>

Commit message: max I@35µm
Parts:
- added E$30: (no value), ucruler:SILK-TABLE-CURRENT-35-TRACE-IPC-2221A
Changed lines of the file:
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@@
 <element name="E$28" library="ucruler" package="SILK-TABLE-THVIA" value="" x="131" y="27" rot="MR0"/>
 <element name="E$29" library="ucruler" package="SILK-TABLE-MM-MIL" value="" x="121" y="29" rot="MR0"/>
+<element name="E$30" library="ucruler" package="SILK-TABLE-CURRENT-35-TRACE-IPC-2221A" value="" x="112.5" y="27" rot="MR0"/>
 </elements>
 <signals>

Commit message: added dpak, d2pak
Parts:
- added E$31: (no value), ucruler:PACK-TO252
- added E$32: (no value), ucruler:PACK-TO263
Other:
- board text added: "TO-252/DPAK"
- board text added: "TO-263/D2PAK"
Changed lines of the file:
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@@
 <setting verticaltext="up"/>
 </settings>
-<grid distance="1" unitdist="mm" unit="mm" style="lines" multiple="1" display="yes" altdistance="0.1" altunitdist="mm" altunit="mm"/>
+<grid distance="0.05" unitdist="inch" unit="mm" style="lines" multiple="1" display="yes" altdistance="0.025" altunitdist="inch" altunit="mm"/>
 <layers>
-<layer number="1" name="Top" color="4" fill="1" visible="no" active="yes"/>
+<layer number="1" name="Top" color="4" fill="1" visible="yes" active="yes"/>
 <layer number="2" name="Route2" color="1" fill="3" visible="no" active="no"/>
 <layer number="3" name="Route3" color="4" fill="3" visible="no" active="no"/>
@@
 <layer number="14" name="Route14" color="1" fill="6" visible="no" active="no"/>
 <layer number="15" name="Route15" color="4" fill="6" visible="no" active="no"/>
-<layer number="16" name="Bottom" color="1" fill="1" visible="yes" active="yes"/>
+<layer number="16" name="Bottom" color="1" fill="1" visible="no" active="yes"/>
 <layer number="17" name="Pads" color="2" fill="1" visible="yes" active="yes"/>
 <layer number="18" name="Vias" color="2" fill="1" visible="yes" active="yes"/>
@@
 <layer number="20" name="Dimension" color="15" fill="1" visible="yes" active="yes"/>
 <layer number="21" name="tPlace" color="7" fill="1" visible="yes" active="yes"/>
-<layer number="22" name="bPlace" color="7" fill="1" visible="yes" active="yes"/>
-<layer number="23" name="tOrigins" color="15" fill="1" visible="no" active="yes"/>
-<layer number="24" name="bOrigins" color="15" fill="1" visible="yes" active="yes"/>
-<layer number="25" name="tNames" color="7" fill="1" visible="no" active="yes"/>
-<layer number="26" name="bNames" color="7" fill="1" visible="yes" active="yes"/>
-<layer number="27" name="tValues" color="7" fill="1" visible="no" active="yes"/>
-<layer number="28" name="bValues" color="7" fill="1" visible="yes" active="yes"/>
-<layer number="29" name="tStop" color="7" fill="3" visible="no" active="yes"/>
-<layer number="30" name="bStop" color="7" fill="6" visible="yes" active="yes"/>
+<layer number="22" name="bPlace" color="7" fill="1" visible="no" active="yes"/>
+<layer number="23" name="tOrigins" color="15" fill="1" visible="yes" active="yes"/>
+<layer number="24" name="bOrigins" color="15" fill="1" visible="no" active="yes"/>
+<layer number="25" name="tNames" color="7" fill="1" visible="yes" active="yes"/>
+<layer number="26" name="bNames" color="7" fill="1" visible="no" active="yes"/>
+<layer number="27" name="tValues" color="7" fill="1" visible="yes" active="yes"/>
+<layer number="28" name="bValues" color="7" fill="1" visible="no" active="yes"/>
+<layer number="29" name="tStop" color="7" fill="3" visible="yes" active="yes"/>
+<layer number="30" name="bStop" color="7" fill="6" visible="no" active="yes"/>
 <layer number="31" name="tCream" color="7" fill="4" visible="no" active="yes"/>
 <layer number="32" name="bCream" color="7" fill="5" visible="no" active="yes"/>
@@
 <text x="161.5" y="27" size="0.8" layer="22" ratio="10" rot="MR0">DD</text>
 <text x="161.5" y="10.3" size="0.8" layer="22" ratio="10" rot="MR0">SS</text>
+<text x="162.43" y="14.02" size="1.2" layer="21" font="fixed" rot="R270" align="center-right">TO-252/DPAK</text>
+<text x="170.05" y="11.48" size="1.2" layer="21" font="fixed" rot="R270" align="center-right">TO-263/D2PAK</text>
 </plain>
 <attributes>
@@
 <element name="E$29" library="ucruler" package="SILK-TABLE-MM-MIL" value="" x="121" y="29" rot="MR0"/>
 <element name="E$30" library="ucruler" package="SILK-TABLE-CURRENT-35-TRACE-IPC-2221A" value="" x="112.5" y="27" rot="MR0"/>
+<element name="E$31" library="ucruler" package="PACK-TO252" value="" x="157.48" y="17.78"/>
+<element name="E$32" library="ucruler" package="PACK-TO263" value="" x="168.91" y="7.62" rot="R90"/>
 </elements>
 <signals>

Commit message: SMA, SMB, SMC
Parts:
- added E$33: (no value), ucruler:PACK-DO214AA-SMB
- added E$34: (no value), ucruler:PACK-DO214AB-SMC
- added E$35: (no value), ucruler:PACK-DO214AC-SMA
Changed lines of the file:
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@@
 <element name="E$31" library="ucruler" package="PACK-TO252" value="" x="157.48" y="17.78"/>
 <element name="E$32" library="ucruler" package="PACK-TO263" value="" x="168.91" y="7.62" rot="R90"/>
+<element name="E$33" library="ucruler" package="PACK-DO214AA-SMB" value="" x="133.35" y="20.32" rot="R90"/>
+<element name="E$34" library="ucruler" package="PACK-DO214AB-SMC" value="" x="133.35" y="13.97" rot="R90"/>
+<element name="E$35" library="ucruler" package="PACK-DO214AC-SMA" value="" x="133.35" y="24.13" rot="R90"/>
 </elements>
 <signals>

Commit message: melf, minimelf, micromelf
Parts:
- added E$36: (no value), ucruler:PACK-MELF
- added E$37: (no value), ucruler:PACK-MELF-MINI
- added E$38: (no value), ucruler:PACK-MELF-MICRO
Changed lines of the file:
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@@
 <element name="E$34" library="ucruler" package="PACK-DO214AB-SMC" value="" x="133.35" y="13.97" rot="R90"/>
 <element name="E$35" library="ucruler" package="PACK-DO214AC-SMA" value="" x="133.35" y="24.13" rot="R90"/>
+<element name="E$36" library="ucruler" package="PACK-MELF" value="" x="123.19" y="24.13" rot="R90"/>
+<element name="E$37" library="ucruler" package="PACK-MELF-MINI" value="" x="123.19" y="21.59" rot="R90"/>
+<element name="E$38" library="ucruler" package="PACK-MELF-MICRO" value="" x="123.19" y="19.05" rot="R90"/>
 </elements>
 <signals>

Commit message: plcc4, plcc6
Parts:
- added E$39: (no value), ucruler:PACK-PLCC-4
- added E$40: (no value), ucruler:PACK-PLCC-6
Changed lines of the file:
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@@
 <element name="E$37" library="ucruler" package="PACK-MELF-MINI" value="" x="123.19" y="21.59" rot="R90"/>
 <element name="E$38" library="ucruler" package="PACK-MELF-MICRO" value="" x="123.19" y="19.05" rot="R90"/>
+<element name="E$39" library="ucruler" package="PACK-PLCC-4" value="" x="123.19" y="15.24" rot="R90"/>
+<element name="E$40" library="ucruler" package="PACK-PLCC-6" value="" x="123.19" y="10.16"/>
 </elements>
 <signals>

Commit message: 0201-1210
Parts:
- added E$41: (no value), ucruler:PACK-0201
- added E$42: (no value), ucruler:PACK-0402
- added E$43: (no value), ucruler:PACK-0603
- added E$44: (no value), ucruler:PACK-0805
- added E$45: (no value), ucruler:PACK-1206
- added E$46: (no value), ucruler:PACK-1210
Changed lines of the file:
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@@
 <element name="E$39" library="ucruler" package="PACK-PLCC-4" value="" x="123.19" y="15.24" rot="R90"/>
 <element name="E$40" library="ucruler" package="PACK-PLCC-6" value="" x="123.19" y="10.16"/>
+<element name="E$41" library="ucruler" package="PACK-0201" value="" x="57.15" y="25.4"/>
+<element name="E$42" library="ucruler" package="PACK-0402" value="" x="57.15" y="24.13"/>
+<element name="E$43" library="ucruler" package="PACK-0603" value="" x="57.15" y="22.86"/>
+<element name="E$44" library="ucruler" package="PACK-0805" value="" x="57.15" y="20.32"/>
+<element name="E$45" library="ucruler" package="PACK-1206" value="" x="57.15" y="17.78"/>
+<element name="E$46" library="ucruler" package="PACK-1210" value="" x="57.15" y="13.97"/>
 </elements>
 <signals>
